Commit message: add meshes for faster examples

File: configs/urdf/heri_II.urdf (robot description, URDF)
Before this commit: robot heri_II, 25 links, 24 joints
Links:
- link LFB1: geometry collision mesh filename=package://end_effector/configs/meshes/heri_II/LFB1.STL; visual mesh filename=package://end_effector/configs/meshes/heri_II/LFB1.STL
- link LFB2: geometry collision mesh filename=package://end_effector/configs/meshes/heri_II/LFB2.STL; visual mesh filename=package://end_effector/configs/meshes/heri_II/LFB2.STL
- link LFB3: geometry collision mesh filename=package://end_effector/configs/meshes/heri_II/LFB3.STL; visual mesh filename=package://end_effector/configs/meshes/heri_II/LFB3.STL
- link LFP1_1: geometry collision mesh filename=package://end_effector/configs/meshes/heri_II/LFP1_1.STL; visual mesh filename=package://end_effector/configs/meshes/heri_II/LFP1_1.STL
- link LFP1_2: geometry collision mesh filename=package://end_effector/configs/meshes/heri_II/LFP1_2.STL; visual mesh filename=package://end_effector/configs/meshes/heri_II/LFP1_2.STL
- link LFP1_3: geometry collision mesh filename=package://end_effector/configs/meshes/heri_II/LFP1_3.STL; visual mesh filename=package://end_effector/configs/meshes/heri_II/LFP1_3.STL
- link LFP2_1: geometry collision mesh filename=package://end_effector/configs/meshes/heri_II/LFP2_1.STL; visual mesh filename=package://end_effector/configs/meshes/heri_II/LFP2_1.STL
- link LFP2_2: geometry collision mesh filename=package://end_effector/configs/meshes/heri_II/LFP2_2.STL; visual mesh filename=package://end_effector/configs/meshes/heri_II/LFP2_2.STL
- link LFP2_3: geometry collision mesh filename=package://end_effector/configs/meshes/heri_II/LFP2_3.STL; visual mesh filename=package://end_effector/configs/meshes/heri_II/LFP2_3.STL
- link LFP3_1: geometry collision mesh filename=package://end_effector/configs/meshes/heri_II/LFP3_1.STL; visual mesh filename=package://end_effector/configs/meshes/heri_II/LFP3_1.STL
- link LFP3_2: geometry collision mesh filename=package://end_effector/configs/meshes/heri_II/LFP3_2.STL; visual mesh filename=package://end_effector/configs/meshes/heri_II/LFP3_2.STL
- link LFP3_3: geometry collision mesh filename=package://end_effector/configs/meshes/heri_II/LFP3_3.STL; visual mesh filename=package://end_effector/configs/meshes/heri_II/LFP3_3.STL
- link SFB1: geometry collision mesh filename=package://end_effector/configs/meshes/heri_II/SFB1.STL; visual mesh filename=package://end_effector/configs/meshes/heri_II/SFB1.STL
- link SFB1_1: geometry collision mesh filename=package://end_effector/configs/meshes/heri_II/SFB1_1.STL; visual mesh filename=package://end_effector/configs/meshes/heri_II/SFB1_1.STL
- link SFP1_2: geometry collision mesh filename=package://end_effector/configs/meshes/heri_II/SFP1_2.STL; visual mesh filename=package://end_effector/configs/meshes/heri_II/SFP1_2.STL
- link base_link: geometry collision mesh filename=package://end_effector/configs/meshes/heri_II/base_heri_ii.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; visual mesh filename=package://end_effector/configs/meshes/heri_II/base_heri_ii.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
Joints:
- joint motor_finger1: limit lower=0 upper=2.5 effort=10 velocity=1 -> lower=0 upper=0.9 effort=10 velocity=1
- joint motor_finger2: limit lower=0 upper=2.5 effort=10 velocity=1 -> lower=0 upper=0.9 effort=10 velocity=1
- joint motor_finger3: limit lower=0 upper=2.5 effort=10 velocity=1 -> lower=0 upper=0.9 effort=10 velocity=1
- joint motor_thumb: limit lower=0 upper=2 effort=10 velocity=1 -> lower=0 upper=1.3 effort=10 velocity=1

File: configs/urdf/schunk.urdf (robot description, URDF)
Before this commit: robot schunk, 32 links, 31 joints
Links:
- link left_hand_a: geometry collision mesh filename=package://end_effector/configs/meshes/d11.dae scale=1 -1 -1; visual mesh filename=package://end_effector/configs/meshes/d11.dae scale=1 -1 -1
- link left_hand_b: geometry collision mesh filename=package://end_effector/configs/meshes/d12.dae scale=1 -1 -1; visual mesh filename=package://end_effector/configs/meshes/d12.dae scale=1 -1 -1
- link left_hand_base_link: geometry collision mesh filename=package://end_effector/configs/meshes/base10.dae; visual mesh filename=package://end_effector/configs/meshes/base10.dae
- link left_hand_c: geometry collision mesh filename=package://end_effector/configs/meshes/d13.dae scale=1 -1 -1; visual mesh filename=package://end_effector/configs/meshes/d13.dae scale=1 -1 -1
- link left_hand_e1: geometry collision mesh filename=package://end_effector/configs/meshes/h10.dae scale=-1 1 1; visual mesh filename=package://end_effector/configs/meshes/h10.dae scale=-1 1 1
- link left_hand_e2: geometry collision mesh filename=package://end_effector/configs/meshes/h11.dae scale=-1 1 1; visual mesh filename=package://end_effector/configs/meshes/h11.dae scale=-1 1 1
- link left_hand_i: geometry collision mesh filename=package://end_effector/configs/meshes/f41.dae; visual mesh filename=package://end_effector/configs/meshes/f41.dae
- link left_hand_j: geometry collision mesh filename=package://end_effector/configs/meshes/f31.dae; visual mesh filename=package://end_effector/configs/meshes/f31.dae
- link left_hand_k: geometry collision mesh filename=package://end_effector/configs/meshes/f21.dae; visual mesh filename=package://end_effector/configs/meshes/f21.dae
- link left_hand_l: geometry collision mesh filename=package://end_effector/configs/meshes/f11.dae; visual mesh filename=package://end_effector/configs/meshes/f11.dae
- link left_hand_m: geometry collision mesh filename=package://end_effector/configs/meshes/f42.dae; visual mesh filename=package://end_effector/configs/meshes/f42.dae
- link left_hand_n: geometry collision mesh filename=package://end_effector/configs/meshes/f32.dae; visual mesh filename=package://end_effector/configs/meshes/f32.dae
- link left_hand_o: geometry collision mesh filename=package://end_effector/configs/meshes/f22.dae; visual mesh filename=package://end_effector/configs/meshes/f22.dae
- link left_hand_p: geometry collision mesh filename=package://end_effector/configs/meshes/f12.dae; visual mesh filename=package://end_effector/configs/meshes/f12.dae
- link left_hand_q: geometry collision mesh filename=package://end_effector/configs/meshes/f43.dae; visual mesh filename=package://end_effector/configs/meshes/f43.dae
- link left_hand_r: geometry collision mesh filename=package://end_effector/configs/meshes/f33.dae; visual mesh filename=package://end_effector/configs/meshes/f33.dae
- link left_hand_s: geometry collision mesh filename=package://end_effector/configs/meshes/f23.dae; visual mesh filename=package://end_effector/configs/meshes/f23.dae
- link left_hand_t: geometry collision mesh filename=package://end_effector/configs/meshes/f13.dae; visual mesh filename=package://end_effector/configs/meshes/f13.dae
- link left_hand_virtual_i: geometry collision mesh filename=package://end_effector/configs/meshes/f40.dae; visual mesh filename=package://end_effector/configs/meshes/f40.dae
- link left_hand_virtual_j: geometry collision mesh filename=package://end_effector/configs/meshes/f30.dae; visual mesh filename=package://end_effector/configs/meshes/f30.dae
- link left_hand_virtual_k: geometry collision mesh filename=package://end_effector/configs/meshes/f20.dae; visual mesh filename=package://end_effector/configs/meshes/f20.dae
- link left_hand_virtual_l: geometry collision mesh filename=package://end_effector/configs/meshes/f10.dae; visual mesh filename=package://end_effector/configs/meshes/f10.dae
- link left_hand_z: geometry collision mesh filename=package://end_effector/configs/meshes/d10.dae scale=1 -1 1; visual mesh filename=package://end_effector/configs/meshes/d10.dae scale=1 -1 1
